File: ecad/mushroom-backplane-tps54560/mushroom-backplane-tps54560.kicad_pcb (KiCad board)
At the start: 2 copper layers, 24 x 63 mm, 42 parts, among them J1 BUSOUT, J2 BUSIN, J3 BACKPLANE, M1 KK 254, Q1 AO3400A, Q2 SI2301CDS-T1-GE3, U1 TPS54560

Commit message: Align pin numbering of backplane and blade
Parts:
- moved J3 15.5 mm to (107.5, 130.2), turned to 270 degrees
Connections:
- J3 pad 10: FANDCC -> FANPWM
- J3 pad 12: SCL -> SDA
- J3 pad 3: SDA -> SCL
- J3 pad 5: FANPWM -> FANDCC
- J3 pad 6: STX -> SRX
- J3 pad 7: FANFDB -> POWTMP
- J3 pad 8: POWTMP -> FANFDB
- J3 pad 9: SRX -> STX
